Commit message: Add data communication

File: install/sjtu_drone_description/share/sjtu_drone_description/urdf/sjtu_drone.urdf (robot description, URDF)
Before this commit: robot sjtu_drone, 5 links, 4 joints
Links:
- link base_link: geometry collision mesh filename=file:///home/widha893/ros2_hil_quadrotor/install/sjtu_drone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; visual mesh filename=file:///home/widha893/ros2_hil_quadrotor/install/sjtu_drone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

File: install/sjtu_drone_description/share/sjtu_drone_description/urdf/sjtu_drone.urdf.xacro (robot description, xacro)
@@ -136,8 +136,8 @@
         <scan>
           <horizontal>
-            <samples>5</samples>
+            <samples>1</samples>
             <resolution>1.000000</resolution>
-            <min_angle>-0.12</min_angle>
-            <max_angle>0.12</max_angle>
+            <min_angle>0</min_angle>
+            <max_angle>0</max_angle>
           </horizontal>
           <vertical>
